Commit message: 初始化项目-CASBOT02硬限位零位测试-web端

File: src/zero_offset_calibration/casbot_band_urdf/urdf/CASBOT02_ENCOS_7dof_shell_20251015_P1L_bass.urdf (robot description, URDF)
Before this commit: robot CB02_URDF(ECS)130C, 59 links, 58 joints
Links:
- link waist_yaw_link: geometry collision mesh filename=../meshes/waist_yaw_link_bass.STL; visual mesh filename=../meshes/waist_yaw_link_bass.STL
Joints:
- joint left_elbow_pitch_joint: limit lower=-2.268 upper=0 effort=75 velocity=12.2 -> lower=-2.26893 upper=0.34907 effort=75 velocity=12.2
- joint left_shoulder_pitch_joint: limit lower=-3.1416 upper=1.0472 effort=75 velocity=12.2 -> lower=-3.22886 upper=1.60570 effort=75 velocity=12.2
- joint left_shoulder_roll_joint: limit lower=-0.3491 upper=3.1416 effort=75 velocity=12.2 -> lower=-0.34906585 upper=3.14159265 effort=75 velocity=12.2
- joint right_elbow_pitch_joint: limit lower=-2.268 upper=0 effort=75 velocity=12.2 -> lower=-2.26893 upper=0.34907 effort=75 velocity=12.2
- joint right_shoulder_pitch_joint: limit lower=-3.1416 upper=1.0472 effort=75 velocity=12.2 -> lower=-3.22886 upper=1.60570 effort=75 velocity=12.2
- joint right_shoulder_roll_joint: limit lower=-3.1416 upper=0.3491 effort=75 velocity=12.2 -> lower=-3.14159265 upper=0.34906585 effort=75 velocity=12.2
- joint right_shoulder_yaw_joint: limit lower=-1.5708 upper=1.5708 effort=36 velocity=9.3 -> lower=-1.57079633 upper=1.57079633 effort=36 velocity=9.3
- joint right_wrist_pitch_joint: limit lower=-1.0472 upper=1.0472 effort=36 velocity=9.3 -> lower=-1.04719755 upper=1.04719755 effort=36 velocity=9.3
- joint right_wrist_roll_joint: limit lower=-1.0472 upper=1.5708 effort=36 velocity=9.3 -> lower=-1.04719755 upper=1.57079633 effort=36 velocity=9.3
- joint right_wrist_yaw_joint: limit lower=-1.5708 upper=1.5708 effort=36 velocity=9.3 -> lower=-1.57079633 upper=1.57079633 effort=36 velocity=9.3
